Commit message: fix: restore custom right MCP2 limits

File: assets/custom_right/URDF_R.urdf (robot description, URDF)
Before this commit: robot URDF_0605_R, 24 links, 23 joints
Joints:
- joint F2-R-MCP2: limit lower=-0.024546 upper=0.349248 effort=6.0 velocity=3.59 -> lower=-0.61 upper=0.61 effort=6.0 velocity=3.59
- joint F3-R-MCP2: limit lower=-0.125311 upper=0.183063 effort=6.0 velocity=3.59 -> lower=-0.61 upper=0.61 effort=6.0 velocity=3.59
- joint F4-R-MCP2: limit lower=-0.134074 upper=0.065926 effort=6.0 velocity=3.59 -> lower=-0.61 upper=0.61 effort=6.0 velocity=3.59
- joint F5-R-MCP2: limit lower=-0.30 upper=0.35 effort=6.0 velocity=3.59 -> lower=-0.61 upper=0.61 effort=6.0 velocity=3.59
