Commit message: 修改了左右手costom hand的AA默认初始位置

File: assets/custom_left/URDF_L.urdf (robot description, URDF)
Before this commit: robot URDF_0605_L, 24 links, 23 joints
Joints:
- joint F2-L-MCP2: origin xyz=0.04512 0.078019 0.00395 rpy=3.1416 0 3.1416 -> xyz=0.04512 0.078019 0.00395 rpy=3.1416 0 2.8798
- joint F4-L-MCP2: origin xyz=0.0059875 0.078019 0.00395 rpy=3.1416 0 3.1416 -> xyz=0.0059875 0.078019 0.00395 rpy=3.1416 0 3.4034
- joint F5-L-MCP2: origin xyz=-0.01361 0.063366 0.00395 rpy=3.1416 0 3.1416 -> xyz=-0.01361 0.063366 0.00395 rpy=3.1416 0 3.7347

File: assets/custom_right/URDF_R.urdf (robot description, URDF)
Before this commit: robot URDF_0605_R, 24 links, 23 joints
Joints:
- joint F2-R-MCP2: origin xyz=0.0475313 0.0778613 0.0023 rpy=0 0 0 -> xyz=0.0475313 0.0778613 0.0023 rpy=0 0 -0.2618
- joint F4-R-MCP2: origin xyz=0.008399 0.0778613 0.0023 rpy=0 0 0 -> xyz=0.008399 0.0778613 0.0023 rpy=0 0 0.2618
- joint F5-R-MCP2: origin xyz=-0.0111988 0.0632092 0.0023 rpy=0 0 0 -> xyz=-0.0111988 0.0632092 0.0023 rpy=0 0 0.5934

Commit message: 修改了costum hand的限位为原始限位

File: assets/custom_left/URDF_L.urdf (robot description, URDF)
Before this commit: robot URDF_0605_L, 24 links, 23 joints
Joints:
- joint F2-L-MCP2: limit lower=-0.024546 upper=0.349248 effort=6.0 velocity=3.59 -> lower=-0.61 upper=0.61 effort=6.0 velocity=3.59
- joint F3-L-MCP2: limit lower=-0.125311 upper=0.183063 effort=6.0 velocity=3.59 -> lower=-0.61 upper=0.61 effort=6.0 velocity=3.59
- joint F4-L-MCP2: limit lower=-0.134074 upper=0.065926 effort=6.0 velocity=3.59 -> lower=-0.61 upper=0.61 effort=6.0 velocity=3.59
- joint F5-L-MCP2: limit lower=-0.30 upper=0.35 effort=6.0 velocity=3.59 -> lower=-0.61 upper=0.61 effort=6.0 velocity=3.59
- joint PALM-L: limit lower=-1.22 upper=1.22 effort=10.0 velocity=2.5 -> lower=-1.3963 upper=1.0472 effort=10.0 velocity=2.5
- joint WRIST-PALM-L: limit lower=-0.785 upper=0.785 effort=12.0 velocity=2.0 -> lower=-0.6981 upper=0.6981 effort=12.0 velocity=2.0

File: assets/custom_right/URDF_R.urdf (robot description, URDF)
Before this commit: robot URDF_0605_R, 24 links, 23 joints
Joints:
- joint F1-R-MCP2: limit lower=-0.35 upper=0.61 effort=6.5 velocity=2.82 -> lower=-0.3491 upper=0.61 effort=6.5 velocity=2.82
- joint PALM-R: limit lower=-1.22 upper=1.22 effort=10.0 velocity=2.5 -> lower=-1.3963 upper=1.0472 effort=10.0 velocity=2.5
- joint WRIST-PALM-R: limit lower=-0.785 upper=0.785 effort=12.0 velocity=2.0 -> lower=-0.6981 upper=0.6981 effort=12.0 velocity=2.0

Commit message: Train anchor v4 right hand checkpoint

File: assets/custom_left/URDF_L.urdf (robot description, URDF)
Before this commit: robot URDF_0605_L, 24 links, 23 joints
Joints:
- joint F2-L-MCP2: limit lower=-0.61 upper=0.61 effort=6.0 velocity=3.59 -> lower=-0.178025 upper=0.321995 effort=6.0 velocity=3.59
- joint F3-L-MCP2: limit lower=-0.61 upper=0.61 effort=6.0 velocity=3.59 -> lower=-0.250044 upper=0.207785 effort=6.0 velocity=3.59
- joint F4-L-MCP2: limit lower=-0.61 upper=0.61 effort=6.0 velocity=3.59 -> lower=-0.277712 upper=0.239799 effort=6.0 velocity=3.59
- joint F5-L-MCP2: limit lower=-0.61 upper=0.61 effort=6.0 velocity=3.59 -> lower=-0.291557 upper=0.294569 effort=6.0 velocity=3.59

File: assets/custom_right/URDF_R.urdf (robot description, URDF)
Before this commit: robot URDF_0605_R, 24 links, 23 joints
Joints:
- joint F2-R-MCP2: limit lower=-0.61 upper=0.61 effort=6.0 velocity=3.59 -> lower=-0.147353 upper=0.32864 effort=6.0 velocity=3.59
- joint F3-R-MCP2: limit lower=-0.61 upper=0.61 effort=6.0 velocity=3.59 -> lower=-0.280029 upper=0.279485 effort=6.0 velocity=3.59
- joint F4-R-MCP2: limit lower=-0.61 upper=0.61 effort=6.0 velocity=3.59 -> lower=-0.247702 upper=0.318512 effort=6.0 velocity=3.59
- joint F5-R-MCP2: limit lower=-0.61 upper=0.61 effort=6.0 velocity=3.59 -> lower=-0.3 upper=0.265075 effort=6.0 velocity=3.59

Commit message: Add manual closure prior to AA limit search

File: assets/custom_left/URDF_L.urdf (robot description, URDF)
Before this commit: robot URDF_0605_L, 24 links, 23 joints
Joints:
- joint F2-L-MCP2: limit lower=-0.178025 upper=0.321995 effort=6.0 velocity=3.59 -> lower=-0.3 upper=0.344806 effort=6.0 velocity=3.59
- joint F3-L-MCP2: limit lower=-0.250044 upper=0.207785 effort=6.0 velocity=3.59 -> lower=-0.166002 upper=0.124275 effort=6.0 velocity=3.59
- joint F4-L-MCP2: limit lower=-0.277712 upper=0.239799 effort=6.0 velocity=3.59 -> lower=-0.3 upper=0.201738 effort=6.0 velocity=3.59
- joint F5-L-MCP2: limit lower=-0.291557 upper=0.294569 effort=6.0 velocity=3.59 -> lower=-0.243689 upper=0.240955 effort=6.0 velocity=3.59

File: assets/custom_right/URDF_R.urdf (robot description, URDF)
Before this commit: robot URDF_0605_R, 24 links, 23 joints
Joints:
- joint F2-R-MCP2: limit lower=-0.147353 upper=0.32864 effort=6.0 velocity=3.59 -> lower=-0.176905 upper=0.35 effort=6.0 velocity=3.59
- joint F3-R-MCP2: limit lower=-0.280029 upper=0.279485 effort=6.0 velocity=3.59 -> lower=-0.228696 upper=0.334765 effort=6.0 velocity=3.59
- joint F4-R-MCP2: limit lower=-0.247702 upper=0.318512 effort=6.0 velocity=3.59 -> lower=-0.299815 upper=0.283408 effort=6.0 velocity=3.59
- joint F5-R-MCP2: limit lower=-0.3 upper=0.265075 effort=6.0 velocity=3.59 -> lower=-0.270761 upper=0.25782 effort=6.0 velocity=3.59

Commit message: Store final custom hand checkpoints

File: assets/custom_left/URDF_L.urdf (robot description, URDF)
Before this commit: robot URDF_0605_L, 24 links, 23 joints
Joints:
- joint F2-L-MCP2: limit lower=-0.3 upper=0.344806 effort=6.0 velocity=3.59 -> lower=-0.380431 upper=0.087049 effort=6.0 velocity=3.59
- joint F3-L-MCP2: limit lower=-0.166002 upper=0.124275 effort=6.0 velocity=3.59 -> lower=-0.242572 upper=0.204627 effort=6.0 velocity=3.59
- joint F4-L-MCP2: limit lower=-0.3 upper=0.201738 effort=6.0 velocity=3.59 -> lower=-0.498692 upper=0.477526 effort=6.0 velocity=3.59
- joint F5-L-MCP2: limit lower=-0.243689 upper=0.240955 effort=6.0 velocity=3.59 -> lower=-0.440455 upper=0.61 effort=6.0 velocity=3.59

File: assets/custom_right/URDF_R.urdf (robot description, URDF)
Before this commit: robot URDF_0605_R, 24 links, 23 joints
Joints:
- joint F2-R-MCP2: limit lower=-0.176905 upper=0.35 effort=6.0 velocity=3.59 -> lower=-0.380431 upper=0.087049 effort=6.0 velocity=3.59
- joint F3-R-MCP2: limit lower=-0.228696 upper=0.334765 effort=6.0 velocity=3.59 -> lower=-0.242572 upper=0.204627 effort=6.0 velocity=3.59
- joint F4-R-MCP2: limit lower=-0.299815 upper=0.283408 effort=6.0 velocity=3.59 -> lower=-0.498692 upper=0.477526 effort=6.0 velocity=3.59
- joint F5-R-MCP2: limit lower=-0.270761 upper=0.25782 effort=6.0 velocity=3.59 -> lower=-0.440455 upper=0.61 effort=6.0 velocity=3.59

Commit message: Restore original custom hand limits before AnyDexRT Step 1

File: assets/custom_left/URDF_L.urdf (robot description, URDF)
Before this commit: robot URDF_0605_L, 24 links, 23 joints
Joints:
- joint F2-L-MCP2: limit lower=-0.380431 upper=0.087049 effort=6.0 velocity=3.59 -> lower=-0.61 upper=0.61 effort=6.0 velocity=3.59
- joint F3-L-MCP2: limit lower=-0.242572 upper=0.204627 effort=6.0 velocity=3.59 -> lower=-0.61 upper=0.61 effort=6.0 velocity=3.59
- joint F4-L-MCP2: limit lower=-0.498692 upper=0.477526 effort=6.0 velocity=3.59 -> lower=-0.61 upper=0.61 effort=6.0 velocity=3.59
- joint F5-L-MCP2: limit lower=-0.440455 upper=0.61 effort=6.0 velocity=3.59 -> lower=-0.61 upper=0.61 effort=6.0 velocity=3.59

File: assets/custom_right/URDF_R.urdf (robot description, URDF)
Before this commit: robot URDF_0605_R, 24 links, 23 joints
Joints:
- joint F2-R-MCP2: limit lower=-0.380431 upper=0.087049 effort=6.0 velocity=3.59 -> lower=-0.61 upper=0.61 effort=6.0 velocity=3.59
- joint F3-R-MCP2: limit lower=-0.242572 upper=0.204627 effort=6.0 velocity=3.59 -> lower=-0.61 upper=0.61 effort=6.0 velocity=3.59
- joint F4-R-MCP2: limit lower=-0.498692 upper=0.477526 effort=6.0 velocity=3.59 -> lower=-0.61 upper=0.61 effort=6.0 velocity=3.59
- joint F5-R-MCP2: limit lower=-0.440455 upper=0.61 effort=6.0 velocity=3.59 -> lower=-0.61 upper=0.61 effort=6.0 velocity=3.59
